File: tbc_ui.kicad_sch (KiCad schematic)
At the start: 39 parts, among them J1 75869-105LF, SW1 PEC11R-4220F-S0024, SW2 TL1100F160Q, U1 CD74HC14M96, U2 ICM7555CBAZ

Commit message: changed 555 to 5V
Connections:
- net +3V3: no longer C7.2, R8.2, U2.4 (~{RESET}), U2.8 (VDD)
- net FREEZE: now also J1.21; no longer J1.22
- new net +5V: C7.2, J1.22, R8.2, U2.4 (~{RESET}), U2.8 (VDD)
- no-connect marks 16 -> 15
